File: camera-hq/raspberry-pi-camera-hq.kicad_pcb (KiCad board)
At the start: 2 copper layers, 38 x 38 mm, 6 parts

Commit message: Update Library
Parts:
- H101, H102, H103, H104: value MountingHole_2.5mm -> 2.5mm
- INFO101: value ORDER-NUMBER -> ~; footprint V2_Production:Order_Number -> V2_Production:Revision
Routing:
- added copper zone on F.Cu, net (none)
- removed copper zone on F.Cu, net GND
