File: camera-hq/raspberry-pi-camera-hq.kicad_sch (KiCad schematic)
At the start: 6 parts

Commit message: Update Library
Parts:
- H101, H102, H103, H104: value MountingHole_2.5mm -> 2.5mm
- INFO101: value ORDER-NUMBER -> ~; footprint V2_Production:Order_Number -> V2_Production:Revision; symbol V2_Production:Order_Number -> V2_Production:Revision
Changed lines of the file:
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@@
 (kicad_sch
-	(version 20231120)
+	(version 20250114)
 	(generator "eeschema")
-	(generator_version "8.0")
+	(generator_version "9.0")
 	(paper "A4")
 	(title_block
 		(title "V2 Rpi Camera HQ")
-		(date "2023-10-11")
-		(rev "1")
+		(date "2026-02-15")
+		(rev "2026-02-15")
 		(company "Versio Duo")
 		(comment 1 "Cover")
@@
 		(at 107.95 66.04 270)
 		(unit 1)
-		(exclude_from_sim yes)
+		(exclude_from_sim no)
 		(in_bom no)
 		(on_board yes)
@@
 			)
 		)
-		(property "Value" "MountingHole_2.5mm"
+		(property "Value" "2.5mm"
 			(at 110.49 67.31 90)
 			(effects
@@
 			)
 		)
-		(property "Description" ""
+		(property "Description" "Mounting Hole without connection"
 			(at 107.95 66.04 0)
 			(effects
@@
 	)
 	(symbol
-		(lib_id "V2_Production:Order_Number")
+		(lib_id "V2_Production:Revision")
 		(at 140.97 109.22 0)
 		(unit 1)
-		(exclude_from_sim yes)
+		(exclude_from_sim no)
 		(in_bom no)
 		(on_board yes)
@@
 			)
 		)
-		(property "Value" "ORDER-NUMBER"
+		(property "Value" "~"
 			(at 140.97 111.76 0)
 			(effects
@@
 			)
 		)
-		(property "Footprint" "V2_Production:Order_Number"
+		(property "Footprint" "V2_Production:Revision"
 			(at 140.97 114.3 0)
 			(effects
@@
 		(at 107.95 81.28 270)
 		(unit 1)
-		(exclude_from_sim yes)
+		(exclude_from_sim no)
 		(in_bom no)
 		(on_board yes)
@@
 			)
 		)
-		(property "Value" "MountingHole_2.5mm"
+		(property "Value" "2.5mm"
 			(at 110.49 82.55 90)
 			(effects
@@
 			)
 		)
-		(property "Description" ""
+		(property "Description" "Mounting Hole without connection"
 			(at 107.95 81.28 0)
 			(effects
@@
 		(at 107.95 58.42 270)
 		(unit 1)
-		(exclude_from_sim yes)
+		(exclude_from_sim no)
 		(in_bom no)
 		(on_board yes)
@@
 			)
 		)
-		(property "Value" "MountingHole_2.5mm"
-			(at 120.65 59.6899 90)
+		(property "Value" "2.5mm"
+			(at 113.792 59.6899 90)
 			(effects
 				(font
@@
 			)
 		)
-		(property "Description" ""
+		(property "Description" "Mounting Hole without connection"
 			(at 107.95 58.42 0)
 			(effects
@@
 		(at 107.95 110.49 0)
 		(unit 1)
-		(exclude_from_sim yes)
+		(exclude_from_sim no)
 		(in_bom no)
 		(on_board yes)
@@
 					(size 1.778 1.5113)
 				)
+				(hide yes)
 			)
 		)
@@
 		(at 107.95 73.66 270)
 		(unit 1)
-		(exclude_from_sim yes)
+		(exclude_from_sim no)
 		(in_bom no)
 		(on_board yes)
@@
 			)
 		)
-		(property "Value" "MountingHole_2.5mm"
+		(property "Value" "2.5mm"
 			(at 110.49 74.93 90)
 			(effects
@@
 			)
 		)
-		(property "Description" ""
+		(property "Description" "Mounting Hole without connection"
 			(at 107.95 73.66 0)
 			(effects
@@
 		)
 	)
+	(embedded_fonts no)
 )
