File: five/raspberry-pi-5.kicad_pcb (KiCad board)
At the start: 4 copper layers, 85 x 56 mm, 47 parts, among them J101 JAE_DX07S016JA3, J104 Raspberry Pi, J201 M.2, J202 SIM, SW101 SW_Push, U101 TPM_Infineon_SLB9670, U501 TPSM33625

Commit message: Update Library
Parts:
- C101, C102, C103, C104, C105, C203, C204, C205, C502, C504: footprint Capacitor_SMD:C_0603_1608Metric -> V2_Capacitor_SMD:C_0603
- C201, C202: footprint Capacitor_Tantalum_SMD:CP_EIA-3528-21_Kemet-B -> V2_Capacitor_SMD:EIA3528
- C501: footprint Capacitor_SMD:C_1210_3225Metric -> V2_Capacitor_SMD:C_1210
- C503, C505: value 22u -> 10u; footprint Capacitor_SMD:C_1210_3225Metric -> V2_Capacitor_SMD:C_1210
- D101, D102, D201: footprint LED_SMD:LED_0603_1608Metric -> V2_LED:LED_0603
- FID101, FID102, FID103: value Fiducial -> Fiducial_Paste
- H101, H102, H103, H104: value MountingHole_2.5mm_PadTop_5mm -> 2.5mm_PadTop_5mm
- INFO101: value ORDER-NUMBER -> ~; footprint V2_Production:Order_Number -> V2_Production:Revision
- J101: value JAE_DX07S016JA3 -> DX07S016JA3
- J104: value Raspberry Pi -> ~
- J201: value M.2 -> ~
- J202: value SIM -> G85D1171012HHR
- R101, R102, R103, R104, R106, R201, R202, R501, R502: footprint Resistor_SMD:R_0603_1608Metric -> V2_Resistor_SMD:R_0603
- R105: value 5K1 -> 5k1; footprint Resistor_SMD:R_0603_1608Metric -> V2_Resistor_SMD:R_0603
- SW101: value SW_Push -> SKSG
- U501: footprint V2_Converter_DCDC:TPSM33625 -> V2_Converter_DCDC:QFN-11
- renumbered H105 to RP105
Connections:
- net +3.3V renamed +3V3
- net Earth renamed Shield
