File: five/raspberry-pi-5.kicad_pcb (KiCad board)
At the start: 4 copper layers, 85 x 56 mm, 47 parts, among them J101 DX07S016JA3, J202 G85D1171012HHR, SW101 SKSG, U101 TPM_Infineon_SLB9670, U501 TPSM33625

Commit message: Replace step-down
Parts:
- U501: value TPSM33625 -> TPSM33620S5QRDNRQ1
Connections:
- U501 pad 11: /Power Supply +3V8/Vcc -> GND
Routing:
- net /Power Supply +3V8/Vcc: track 9.71 -> 1.64 mm
- net GND: track 44.4 -> 42.0 mm, vias 68 -> 70
