File: five/M2-Connector.kicad_sch (KiCad schematic)
At the start: 13 parts, among them J101 JAE_DX07S016JA3, J201 M.2, J202 SIM

Commit message: Update Library
Parts:
- C201, C202: footprint Capacitor_Tantalum_SMD:CP_EIA-3528-21_Kemet-B -> V2_Capacitor_SMD:EIA3528; symbol Device:C_Polarized_Small -> V2_Capacitor:Polarized_EIA3528_100u; Manufacturer (none) -> KEMET; Mouser (none) -> 80-T491B107K006; Product (none) -> T491B107K006AT
- C203, C204, C205: footprint Capacitor_SMD:C_0603_1608Metric -> V2_Capacitor_SMD:C_0603; symbol Device:C_Small -> V2_Capacitor:0603_0u1; Manufacturer (none) -> TDK; Mouser (none) -> 810-CGA3E2X7R1H104MA; Product (none) -> CGA3E2X7R1H104M080AA; Rating (none) -> 50V
- D201: footprint LED_SMD:LED_0603_1608Metric -> V2_LED:LED_0603; symbol Device:LED_Small -> V2_LED:0603_Orange; Manufacturer (none) -> ROHM Semiconductor; Mouser (none) -> 755-SML-D12D1WT86; Product (none) -> SML-D12D1WT86
- J101: value JAE_DX07S016JA3 -> DX07S016JA3; Manufacturer (none) -> JAE Electronics; Mouser (none) -> 656-DX07S016JA3R1500; Product (none) -> DX07S016JA3R1500
- J201: value M.2 -> ~
- J202: value SIM -> G85D1171012HHR
- R101, R102: footprint Resistor_SMD:R_0603_1608Metric -> V2_Resistor_SMD:R_0603; symbol Device:R_Small -> V2_Resistor:0603_5k1; Manufacturer (none) -> Vishay; Mouser (none) -> 71-CRCW06035K10FKEAC; Product (none) -> CRCW06035K10FKEAC; Rating (none) -> 100mW
- R201: footprint Resistor_SMD:R_0603_1608Metric -> V2_Resistor_SMD:R_0603; symbol Device:R_Small -> V2_Resistor:0603_1k; Manufacturer (none) -> Vishay; Mouser (none) -> 71-CRCW06031K00FKEAH; Product (none) -> CRCW06031K00FKEAHP; Rating (none) -> 330mW
- R202: footprint Resistor_SMD:R_0603_1608Metric -> V2_Resistor_SMD:R_0603; symbol Device:R_Small -> V2_Resistor:0603_27k
Connections:
- net Earth renamed Shield

Commit message: KiCad 10
Parts:
- J201: value ~ -> (none)

Commit message: Good Bye Imperial
Parts:
- C203, C204, C205: footprint V2_Capacitor_SMD:C_0603 -> V2_Capacitor_SMD:C_1608; symbol V2_Capacitor:0603_0u1 -> V2_Capacitor:1608_0u1
- D201: symbol V2_LED:0603_Orange -> V2_LED:1608_Orange
- R101, R102: footprint V2_Resistor_SMD:R_0603 -> V2_Resistor_SMD:R_1608; symbol V2_Resistor:0603_5k1 -> V2_Resistor:1608_5k1
- R201: footprint V2_Resistor_SMD:R_0603 -> V2_Resistor_SMD:R_1608; symbol V2_Resistor:0603_1k -> V2_Resistor:1608_1k
- R202: footprint V2_Resistor_SMD:R_0603 -> V2_Resistor_SMD:R_1608; symbol V2_Resistor:0603_27k -> V2_Resistor:1608_27k
Changed lines of the file:
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@@
 	)
 	(symbol
-		(lib_id "V2_Resistor:0603_5k1")
+		(lib_id "V2_Resistor:1608_5k1")
 		(at 80.01 95.25 90)
 		(unit 1)
@@
 			)
 		)
-		(property "Footprint" "V2_Resistor_SMD:R_0603"
+		(property "Footprint" "V2_Resistor_SMD:R_1608"
 			(at 95.758 95.25 0)
 			(hide yes)
@@
 	)
 	(symbol
-		(lib_id "V2_Resistor:0603_1k")
+		(lib_id "V2_Resistor:1608_1k")
 		(at 172.72 63.5 90)
 		(unit 1)
@@
 			)
 		)
-		(property "Footprint" "V2_Resistor_SMD:R_0603"
+		(property "Footprint" "V2_Resistor_SMD:R_1608"
 			(at 188.468 63.5 0)
 			(hide yes)
@@
 	)
 	(symbol
-		(lib_id "V2_Capacitor:0603_0u1")
+		(lib_id "V2_Capacitor:1608_0u1")
 		(at 257.81 87.63 0)
 		(unit 1)
@@
 			)
 		)
-		(property "Footprint" "V2_Capacitor_SMD:C_0603"
+		(property "Footprint" "V2_Capacitor_SMD:C_1608"
 			(at 257.81 104.648 0)
 			(hide yes)
@@
 	)
 	(symbol
-		(lib_id "V2_LED:0603_Orange")
+		(lib_id "V2_LED:1608_Orange")
 		(at 166.37 63.5 0)
 		(mirror x)
@@
 	)
 	(symbol
-		(lib_id "V2_Resistor:0603_5k1")
+		(lib_id "V2_Resistor:1608_5k1")
 		(at 80.01 92.71 90)
 		(unit 1)
@@
 			)
 		)
-		(property "Footprint" "V2_Resistor_SMD:R_0603"
+		(property "Footprint" "V2_Resistor_SMD:R_1608"
 			(at 95.758 92.71 0)
 			(hide yes)
@@
 	)
 	(symbol
-		(lib_id "V2_Capacitor:0603_0u1")
+		(lib_id "V2_Capacitor:1608_0u1")
 		(at 246.38 87.63 0)
 		(unit 1)
@@
 			)
 		)
-		(property "Footprint" "V2_Capacitor_SMD:C_0603"
+		(property "Footprint" "V2_Capacitor_SMD:C_1608"
 			(at 246.38 104.648 0)
 			(hide yes)
@@
 	)
 	(symbol
-		(lib_id "V2_Resistor:0603_27k")
+		(lib_id "V2_Resistor:1608_27k")
 		(at 209.55 114.3 0)
 		(unit 1)
@@
 			)
 		)
-		(property "Footprint" "V2_Resistor_SMD:R_0603"
+		(property "Footprint" "V2_Resistor_SMD:R_1608"
 			(at 209.55 130.048 0)
 			(hide yes)
@@
 	)
 	(symbol
-		(lib_id "V2_Capacitor:0603_0u1")
+		(lib_id "V2_Capacitor:1608_0u1")
 		(at 195.58 87.63 0)
 		(unit 1)
@@
 			)
 		)
-		(property "Footprint" "V2_Capacitor_SMD:C_0603"
+		(property "Footprint" "V2_Capacitor_SMD:C_1608"
 			(at 195.58 104.648 0)
 			(hide yes)
