File: five/raspberry-pi-5-cover/raspberry-pi-5-cover.kicad_pcb (KiCad board)
At the start: 2 copper layers, 85 x 56 mm, 8 parts

Commit message: Update Library
Parts:
- H101, H103, H105, H107: value MountingHole_2.5mm_Pad_5mm -> 2.5mm_Pad_5mm
- INFO101: value ORDER-NUMBER -> ~; footprint V2_Production:Order_Number -> V2_Production:Revision
- renumbered H102 to RP102
Routing:
- net GND: vias 1 -> 0
