File: zero/raspberry-pi-zero.kicad_pcb (KiCad board)
At the start: 4 copper layers, 65 x 30 mm, 30 parts, among them J101 JAE_DX07S016JA3, J102 Pin_2mm, J103 Pin_2mm, J104 Raspberry Pi, SW101 SW_Push, U101 TPM_Infineon_SLB9670

Commit message: Update Library
Parts:
- C101: renamed from C104; footprint Capacitor_SMD:C_0603_1608Metric -> V2_Capacitor_SMD:C_0603
- C102: renamed from C101; footprint Capacitor_SMD:C_0603_1608Metric -> V2_Capacitor_SMD:C_0603
- C103: renamed from C102; footprint Capacitor_SMD:C_0603_1608Metric -> V2_Capacitor_SMD:C_0603
- C104: renamed from C105; footprint Capacitor_SMD:C_0603_1608Metric -> V2_Capacitor_SMD:C_0603
- C105: renamed from C103; footprint Capacitor_SMD:C_0603_1608Metric -> V2_Capacitor_SMD:C_0603
- D101, D102: footprint LED_SMD:LED_0603_1608Metric -> V2_LED:LED_0603
- FID101, FID102, FID103: value Fiducial -> Fiducial_Paste
- H102: renamed from H101; value MountingHole_2.5mm_PadTop_5mm -> 2.5mm_PadTop_5mm
- H103: renamed from H102; value MountingHole_2.5mm_PadTop_5mm -> 2.5mm_PadTop_5mm
- H104: renamed from H103; value MountingHole_2.5mm_PadTop_5mm -> 2.5mm_PadTop_5mm
- H105: renamed from H104; value MountingHole_2.5mm_PadTop_5mm -> 2.5mm_PadTop_5mm
- INFO101: value ORDER-NUMBER -> ~; footprint V2_Production:Order_Number -> V2_Production:Revision
- J101: renamed from J104; value Raspberry Pi -> ~
- J102: renamed from J101; value JAE_DX07S016JA3 -> DX07S016JA3
- R101: renamed from R106; footprint Resistor_SMD:R_0603_1608Metric -> V2_Resistor_SMD:R_0603
- R102: renamed from R105; value 5K1 -> 5k1; footprint Resistor_SMD:R_0603_1608Metric -> V2_Resistor_SMD:R_0603
- R103: renamed from R101; footprint Resistor_SMD:R_0603_1608Metric -> V2_Resistor_SMD:R_0603
- R104: renamed from R102; footprint Resistor_SMD:R_0603_1608Metric -> V2_Resistor_SMD:R_0603
- R105: renamed from R103; footprint Resistor_SMD:R_0603_1608Metric -> V2_Resistor_SMD:R_0603
- R106: renamed from R104; footprint Resistor_SMD:R_0603_1608Metric -> V2_Resistor_SMD:R_0603
- SW101: value SW_Push -> SKSG
- renumbered J102 to J104, H105 to RP101
Connections:
- net +3.3V renamed +3V3
- net Earth renamed Shield
