File: zero/raspberry-pi-zero.kicad_sch (KiCad schematic)
At the start: 30 parts, among them J101 JAE_DX07S016JA3, J102 Pin_2mm, J103 Pin_2mm, J104 Raspberry Pi, SW101 SW_Push, U101 TPM_Infineon_SLB9670

Commit message: Update Library
Parts:
- C101: renamed from C104; footprint Capacitor_SMD:C_0603_1608Metric -> V2_Capacitor_SMD:C_0603; symbol Device:C_Small -> V2_Capacitor:0603_10u; Manufacturer (none) -> TDK; Mouser (none) -> 810-C1608X6S1A106M; Product (none) -> C1608X6S1A106M080AC; Rating (none) -> 10V
- C102: renamed from C101; footprint Capacitor_SMD:C_0603_1608Metric -> V2_Capacitor_SMD:C_0603; symbol Device:C_Small -> V2_Capacitor:0603_0u1; Manufacturer (none) -> TDK; Mouser (none) -> 810-CGA3E2X7R1H104MA; Product (none) -> CGA3E2X7R1H104M080AA; Rating (none) -> 50V
- C103: renamed from C102; footprint Capacitor_SMD:C_0603_1608Metric -> V2_Capacitor_SMD:C_0603; symbol Device:C_Small -> V2_Capacitor:0603_0u1; Manufacturer (none) -> TDK; Mouser (none) -> 810-CGA3E2X7R1H104MA; Product (none) -> CGA3E2X7R1H104M080AA; Rating (none) -> 50V
- C104: renamed from C105; footprint Capacitor_SMD:C_0603_1608Metric -> V2_Capacitor_SMD:C_0603; symbol Device:C_Small -> V2_Capacitor:0603_0u1; Manufacturer (none) -> TDK; Mouser (none) -> 810-CGA3E2X7R1H104MA; Product (none) -> CGA3E2X7R1H104M080AA; Rating (none) -> 50V
- C105: renamed from C103; footprint Capacitor_SMD:C_0603_1608Metric -> V2_Capacitor_SMD:C_0603; symbol Device:C_Small -> V2_Capacitor:0603_0u1; Manufacturer (none) -> TDK; Mouser (none) -> 810-CGA3E2X7R1H104MA; Product (none) -> CGA3E2X7R1H104M080AA; Rating (none) -> 50V
- D101, D102: footprint LED_SMD:LED_0603_1608Metric -> V2_LED:LED_0603; symbol Device:LED_Small -> V2_LED:0603_Orange; Manufacturer (none) -> ROHM Semiconductor; Mouser (none) -> 755-SML-D12D1WT86; Product (none) -> SML-D12D1WT86
- FID101, FID102, FID103: value Fiducial -> Fiducial_Paste
- H102: renamed from H101; value MountingHole_2.5mm_PadTop_5mm -> 2.5mm_PadTop_5mm
- H103: renamed from H102; value MountingHole_2.5mm_PadTop_5mm -> 2.5mm_PadTop_5mm
- H104: renamed from H103; value MountingHole_2.5mm_PadTop_5mm -> 2.5mm_PadTop_5mm
- H105: renamed from H104; value MountingHole_2.5mm_PadTop_5mm -> 2.5mm_PadTop_5mm
- INFO101: value ORDER-NUMBER -> ~; footprint V2_Production:Order_Number -> V2_Production:Revision; symbol V2_Production:Order_Number -> V2_Production:Revision
- J101: renamed from J104; value Raspberry Pi -> ~
- J102: renamed from J101; value JAE_DX07S016JA3 -> DX07S016JA3; Manufacturer (none) -> JAE Electronics; Mouser (none) -> 656-DX07S016JA3R1500; Product (none) -> DX07S016JA3R1500
- R101: renamed from R106; footprint Resistor_SMD:R_0603_1608Metric -> V2_Resistor_SMD:R_0603; symbol Device:R_Small -> V2_Resistor:0603_10k; Manufacturer (none) -> Vishay; Mouser (none) -> 71-CRCW060310K0FKEAC; Product (none) -> CRCW060310K0FKEAC; Rating (none) -> 100mW
- R102: renamed from R105; value 5K1 -> 5k1; footprint Resistor_SMD:R_0603_1608Metric -> V2_Resistor_SMD:R_0603; symbol Device:R_Small -> V2_Resistor:0603_5k1; Manufacturer (none) -> Vishay; Mouser (none) -> 71-CRCW06035K10FKEAC; Product (none) -> CRCW06035K10FKEAC; Rating (none) -> 100mW
- R103: renamed from R101; footprint Resistor_SMD:R_0603_1608Metric -> V2_Resistor_SMD:R_0603; symbol Device:R_Small -> V2_Resistor:0603_5k1; Manufacturer (none) -> Vishay; Mouser (none) -> 71-CRCW06035K10FKEAC; Product (none) -> CRCW06035K10FKEAC; Rating (none) -> 100mW
- R104: renamed from R102; footprint Resistor_SMD:R_0603_1608Metric -> V2_Resistor_SMD:R_0603; symbol Device:R_Small -> V2_Resistor:0603_5k1; Manufacturer (none) -> Vishay; Mouser (none) -> 71-CRCW06035K10FKEAC; Product (none) -> CRCW06035K10FKEAC; Rating (none) -> 100mW
- R105: renamed from R103; footprint Resistor_SMD:R_0603_1608Metric -> V2_Resistor_SMD:R_0603; symbol Device:R_Small -> V2_Resistor:0603_330R; Manufacturer (none) -> Vishay; Mouser (none) -> 71-CRCW0603330RFKEAC; Product (none) -> CRCW0603330RFKEAC; Rating (none) -> 100mW
- R106: renamed from R104; footprint Resistor_SMD:R_0603_1608Metric -> V2_Resistor_SMD:R_0603; symbol Device:R_Small -> V2_Resistor:0603_330R; Manufacturer (none) -> Vishay; Mouser (none) -> 71-CRCW0603330RFKEAC; Product (none) -> CRCW0603330RFKEAC; Rating (none) -> 100mW
- SW101: value SW_Push -> SKSG; symbol Switch:SW_Push -> V2_Switch:SKSG; Manufacturer (none) -> Alps Alpine; Mouser (none) -> 688-SKSGACE010; Product (none) -> SKSGACE010
- renumbered J102 to J104, H105 to RP101
Connections:
- net +3.3V renamed +3V3
- net Earth renamed Shield
Other:
- moved on the sheet: C101, C102, C103, C104, C105, R101, R102, U101

Commit message: Good Bye Imperial
Parts:
- C101: footprint V2_Capacitor_SMD:C_0603 -> V2_Capacitor_SMD:C_1608; symbol V2_Capacitor:0603_10u -> V2_Capacitor:1608_10u
- C102, C103, C104, C105: footprint V2_Capacitor_SMD:C_0603 -> V2_Capacitor_SMD:C_1608; symbol V2_Capacitor:0603_0u1 -> V2_Capacitor:1608_0u1
- D101, D102: symbol V2_LED:0603_Orange -> V2_LED:1608_Orange
- R101: footprint V2_Resistor_SMD:R_0603 -> V2_Resistor_SMD:R_1608; symbol V2_Resistor:0603_10k -> V2_Resistor:1608_10k
- R102, R103, R104: footprint V2_Resistor_SMD:R_0603 -> V2_Resistor_SMD:R_1608; symbol V2_Resistor:0603_5k1 -> V2_Resistor:1608_5k1
- R105, R106: footprint V2_Resistor_SMD:R_0603 -> V2_Resistor_SMD:R_1608; symbol V2_Resistor:0603_330R -> V2_Resistor:1608_330R
Changed lines of the file:
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@@
 	)
 	(symbol
-		(lib_id "V2_LED:0603_Orange")
+		(lib_id "V2_LED:1608_Orange")
 		(at 238.76 46.99 0)
 		(mirror y)
@@
 	)
 	(symbol
-		(lib_id "V2_Resistor:0603_5k1")
+		(lib_id "V2_Resistor:1608_5k1")
 		(at 86.36 78.74 180)
 		(unit 1)
@@
 			)
 		)
-		(property "Footprint" "V2_Resistor_SMD:R_0603"
+		(property "Footprint" "V2_Resistor_SMD:R_1608"
 			(at 86.36 62.992 0)
 			(effects
@@
 	)
 	(symbol
-		(lib_id "V2_Resistor:0603_330R")
+		(lib_id "V2_Resistor:1608_330R")
 		(at 245.11 33.02 90)
 		(unit 1)
@@
 			)
 		)
-		(property "Footprint" "V2_Resistor_SMD:R_0603"
+		(property "Footprint" "V2_Resistor_SMD:R_1608"
 			(at 260.858 33.02 0)
 			(effects
@@
 	)
 	(symbol
-		(lib_id "V2_LED:0603_Orange")
+		(lib_id "V2_LED:1608_Orange")
 		(at 238.76 33.02 0)
 		(mirror y)
@@
 	)
 	(symbol
-		(lib_id "V2_Resistor:0603_5k1")
+		(lib_id "V2_Resistor:1608_5k1")
 		(at 213.36 93.98 90)
 		(unit 1)
@@
 			)
 		)
-		(property "Footprint" "V2_Resistor_SMD:R_0603"
+		(property "Footprint" "V2_Resistor_SMD:R_1608"
 			(at 229.108 93.98 0)
 			(effects
@@
 	)
 	(symbol
-		(lib_id "V2_Capacitor:0603_0u1")
+		(lib_id "V2_Capacitor:1608_0u1")
 		(at 58.42 58.42 0)
 		(unit 1)
@@
 			)
 		)
-		(property "Footprint" "V2_Capacitor_SMD:C_0603"
+		(property "Footprint" "V2_Capacitor_SMD:C_1608"
 			(at 58.42 75.438 0)
 			(effects
@@
 	)
 	(symbol
-		(lib_id "V2_Capacitor:0603_0u1")
+		(lib_id "V2_Capacitor:1608_0u1")
 		(at 78.74 58.42 0)
 		(unit 1)
@@
 			)
 		)
-		(property "Footprint" "V2_Capacitor_SMD:C_0603"
+		(property "Footprint" "V2_Capacitor_SMD:C_1608"
 			(at 78.74 75.438 0)
 			(effects
@@
 	)
 	(symbol
-		(lib_id "V2_Resistor:0603_10k")
+		(lib_id "V2_Resistor:1608_10k")
 		(at 26.67 81.28 270)
 		(unit 1)
@@
 			)
 		)
-		(property "Footprint" "V2_Resistor_SMD:R_0603"
+		(property "Footprint" "V2_Resistor_SMD:R_1608"
 			(at 10.922 81.28 0)
 			(effects
@@
 	)
 	(symbol
-		(lib_id "V2_Capacitor:0603_10u")
+		(lib_id "V2_Capacitor:1608_10u")
 		(at 55.88 125.73 0)
 		(unit 1)
@@
 			)
 		)
-		(property "Footprint" "V2_Capacitor_SMD:C_0603"
+		(property "Footprint" "V2_Capacitor_SMD:C_1608"
 			(at 55.88 142.748 0)
 			(effects
@@
 	)
 	(symbol
-		(lib_id "V2_Capacitor:0603_0u1")
+		(lib_id "V2_Capacitor:1608_0u1")
 		(at 86.36 83.82 0)
 		(unit 1)
@@
 			)
 		)
-		(property "Footprint" "V2_Capacitor_SMD:C_0603"
+		(property "Footprint" "V2_Capacitor_SMD:C_1608"
 			(at 86.36 100.838 0)
 			(effects
@@
 	)
 	(symbol
-		(lib_id "V2_Capacitor:0603_0u1")
+		(lib_id "V2_Capacitor:1608_0u1")
 		(at 68.58 58.42 0)
 		(unit 1)
@@
 			)
 		)
-		(property "Footprint" "V2_Capacitor_SMD:C_0603"
+		(property "Footprint" "V2_Capacitor_SMD:C_1608"
 			(at 68.58 75.438 0)
 			(effects
@@
 	)
 	(symbol
-		(lib_id "V2_Resistor:0603_330R")
+		(lib_id "V2_Resistor:1608_330R")
 		(at 245.11 46.99 90)
 		(unit 1)
@@
 			)
 		)
-		(property "Footprint" "V2_Resistor_SMD:R_0603"
+		(property "Footprint" "V2_Resistor_SMD:R_1608"
 			(at 260.858 46.99 0)
 			(effects
@@
 	)
 	(symbol
-		(lib_id "V2_Resistor:0603_5k1")
+		(lib_id "V2_Resistor:1608_5k1")
 		(at 213.36 91.44 90)
 		(unit 1)
@@
 			)
 		)
-		(property "Footprint" "V2_Resistor_SMD:R_0603"
+		(property "Footprint" "V2_Resistor_SMD:R_1608"
 			(at 229.108 91.44 0)
 			(effects
