File: zero/raspberry-pi-zero-camera-cover/raspberry-pi-zero-camera-cover.kicad_sch (KiCad schematic)
At the start: 11 parts

Commit message: Update Library
Parts:
- H101, H103, H105, H107: value MountingHole_2.5mm_Pad_5mm -> 2.5mm_Pad_5mm
- H102, H104: value MountingHole_2mm_Pad_4mm -> 2mm_Pad_4mm
- H106: value MountingHole_10mm -> 8mm
- INFO101: value ORDER-NUMBER -> ~; footprint V2_Production:Order_Number -> V2_Production:Revision; symbol V2_Production:Order_Number -> V2_Production:Revision
- renumbered H108 to RP108
