File: zero/raspberry-pi-zero-cover/raspberry-pi-zero-cover.kicad_pcb (KiCad board)
At the start: 2 copper layers, 65 x 30 mm, 8 parts

Commit message: Update Library
Parts:
- H101: value Mounting_Hole -> 2.5mm_Pad_5mm
- H102: renamed from H103; value Mounting_Hole -> 2.5mm_Pad_5mm
- H103: renamed from H105; value Mounting_Hole -> 2.5mm_Pad_5mm
- H104: renamed from H107; value Mounting_Hole -> 2.5mm_Pad_5mm
- INFO101: value ORDER-NUMBER -> ~; footprint V2_Production:Order_Number -> V2_Production:Revision
- RP105: renamed from H108; value Val** -> Zero
Routing:
- net GND: vias 1 -> 0
