File: zero/raspberry-pi-zero-cover/raspberry-pi-zero-cover.kicad_sch (KiCad schematic)
At the start: 8 parts

Commit message: Update Library
Parts:
- H101: value MountingHole_2.5mm_Pad_5mm -> 2.5mm_Pad_5mm
- H102: renamed from H103; value MountingHole_2.5mm_Pad_5mm -> 2.5mm_Pad_5mm
- H103: renamed from H105; value MountingHole_2.5mm_Pad_5mm -> 2.5mm_Pad_5mm
- H104: renamed from H107; value MountingHole_2.5mm_Pad_5mm -> 2.5mm_Pad_5mm
- INFO101: value ORDER-NUMBER -> ~; footprint V2_Production:Order_Number -> V2_Production:Revision; symbol V2_Production:Order_Number -> V2_Production:Revision
- renumbered H108 to RP105
Other:
- moved on the sheet: H101, H102, H103, H104, ICON101, INFO101, RP105, SWT101
